File: babelfish.kicad_sch (KiCad schematic)
At the start: 52 parts, among them J1 TYPE-C-31-M-12, J2 Conn_01x02, J3 SWD, J5 IO_A, J6 IO_B, J7 USB_A, U1 NCP1117-3.3_SOT223, U2 W25Q128JVS, U3 RP2040, U4 WS3232ECY, Y1 X322512MSB4SI

Commit message: updates
Parts:
- added J4: Shifter Power, Connector_PinHeader_2.54mm:PinHeader_2x03_P2.54mm_Vertical, symbol Connector_Generic:Conn_02x03_Odd_Even
- added Q1, Q2, Q3, Q4: ~, Package_TO_SOT_SMD:SOT-23-3, symbol Device:Q_NMOS_DGS
- added R12, R13, R14, R15, R16, R17, R18, R19: 10k, Resistor_SMD:R_0402_1005Metric, symbol Device:R_Small
- C22: value C_Small -> 10u; footprint (none) -> Capacitor_SMD:C_0805_2012Metric
- FB1: footprint (none) -> Inductor_SMD:L_0805_2012Metric
- R10, R9: footprint (none) -> Capacitor_SMD:C_0402_1005Metric
- R11, R5: value 27 -> 22
Connections:
- net +3V3: now also R8.2, J4.6 (Pin_6); no longer R8.1
- net GPIO14: now also R5.2
- net GPIO15: now also R11.2
- net GPIO2: no longer J5.4 (Pin_4)
- net GPIO6: no longer J5.2 (Pin_2)
- net RUN: now also R8.1; no longer R8.2
- net VBUS: now also J4.4 (Pin_4)
- net GPIO16 renamed U0_TX_C
- net U0_TX_C: now also Q1.3 (S), R12.2; no longer R5.2
- net GPIO17 renamed U0_RX_C
- net U0_RX_C: now also Q2.3 (S), R14.2; no longer R11.2
- net GPIO20 renamed U0_RX_CH
- net U0_RX_CH: now also Q2.1 (D), R15.2; no longer U3.31 (GPIO20)
- net GPIO21 renamed U0_TX_CH
- net U0_TX_CH: now also Q1.1 (D), R13.2; no longer U3.32 (GPIO21)
- new net: J4.1 (Pin_1), J4.3 (Pin_3), J4.5 (Pin_5)
- new net +3.3V: Q1.2 (G), Q2.2 (G), Q3.2 (G), Q4.2 (G), R12.1, R14.1, R16.1, R18.1
- new net U1_RX_C: Q4.3 (S), R18.2, U3.32 (GPIO21)
- new net U1_RX_CH: J5.2 (Pin_2), Q4.1 (D), R19.2
- new net U1_TX_C: Q3.3 (S), R16.2, U3.31 (GPIO20)
- new net U1_TX_CH: J5.4 (Pin_4), Q3.1 (D), R17.2
- no-connect marks 12 -> 9
Other:
- note added: "Main USB-C"
- note added: "NB: C10 near pin 44"
- note added: "NB: C8 near pin 45"
- note added: "NB: R3/R4 close to RP2040"
- note added: "Power sources: - 5V from Main USB-C or External. Used as VBUS. Buck to 3v3. - 6V+ from VCC. Buck to 5v VBUS and 3v3."
- note added: "TODO: 1. Test PIO-USB host 2. Test level shifter with 3v3?"
- note added: "USB2 USB-A Host"
- note added: "gpio 16,17 and 20,21"
- note removed: "From USB"
- note removed: "IOs"
- note removed: "Make sure C10 is close to pin 44 of RP2040"
- note removed: "Make sure C8 is close to pin 45 of RP2040"
- note removed: "Make sure R3 and R4 are close to RP2040"
- moved on the sheet: C1, C10, C11, C12, C13, C14, C15, C16, C17, C2, C22, C3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
