File: babelfish.kicad_sch (KiCad schematic)
At the start: 59 parts, among them J3 SWD, J4 Shifter Power, J5 IO_A, J7 USB_A, Q1 BSS138, SW1 K2-1156SP-D5SW-05, U1 NCP1117-3.3_SOT223, U2 W25Q128JVS, U3 RP2040, U4 GT-USB-7010ASV, X1 X322512MSB4SI

Commit message: rev2, pre review
Parts:
- removed J4: Shifter Power, Connector_PinHeader_2.54mm:PinHeader_2x03_P2.54mm_Vertical, symbol Connector_Generic:Conn_02x03_Odd_Even
- added C18: 4u7, Capacitor_SMD:C_0603_1608Metric, symbol Device:C_Small
- added C19: 10u, Capacitor_SMD:C_0805_2012Metric, symbol Device:C_Small
- added D2, D4: Red, LED_SMD:LED_0603_1608Metric, symbol Device:LED_Small
- added D5: Blue, LED_SMD:LED_0603_1608Metric, symbol Device:LED_Small
- added D6: 40V/5A, Diode_SMD:D_SOD-323, symbol Device:D_Schottky_Small
- added L1: 4u7, Inductor_SMD:L_1008_2520Metric, symbol Device:L_Small
- added R21, R22, R23: 68, Resistor_SMD:R_0603_1608Metric, symbol Device:R_Small
- added R24: 47k, Resistor_SMD:R_0603_1608Metric, symbol Device:R_Small
- added R25: 15k, Resistor_SMD:R_0603_1608Metric, symbol Device:R_Small
- added R26: 10k, Resistor_SMD:R_0402_1005Metric, symbol Device:R_Small_US
- added U5: LGS6302, lcsc:SOT-23-5_L3.0-W1.6-P0.95-LS2.8-BL, symbol LCSC:LGS6302
- J3: footprint Connector_PinHeader_2.54mm:PinHeader_1x04_P2.54mm_Vertical -> SnapEDA:490107670412
- SW1: value K2-1156SP-D5SW-05 -> K2-1836UQ-C3DW-06; footprint lcsc:SW-SMD_4P-L6.3-W6.2-P4.00-LS9.4-TL -> lcsc:SW-SMD_4P-L2.8-W2.4-P1.60-LS3.0; symbol LCSC:K2-1156SP-D5SW-05 -> LCSC:K2-1836UQ-C3DW-06; LCSC C128948 -> C128935
- U3: renamed from U1; value NCP1117-3.3_SOT223 -> AMS1117-3.3; symbol Regulator_Linear:NCP1117-3.3_SOT223 -> Regulator_Linear:AMS1117-3.3
- renumbered U3 to U1
Connections:
- net SH_REF is gone; now on net VCC_IN: R13.1, R15.1, R17.1, R19.1
- net +3V3: now also C18.1, L1.1, R26.2, U5.5 (VIN)
- net GND: now also SW1.A, C18.2, C19.2, D2.1 (K), D4.1 (K), D5.1 (K), R25.2, U5.2 (GND); no longer SW1.4
- net SWCLK: now also J3.4 (Pin_4); no longer J3.2 (Pin_2)
- net SWD: now also J3.2 (Pin_2); no longer J3.4 (Pin_4)
- net VBUS: no longer C22.1, FB1.2
- net ~{USB_BOOT}: now also SW1.B; no longer SW1.2
- net OSC1: now reaches C2.1, X1.1 (OSC1)
- net OSC1R: now reaches C2.2, R20.1
- net OSC2: now reaches C3.1, X1.3 (OSC2)
- net GPIO10 renamed LED_P_OK
- net LED_P_OK: now also R22.1
- net GPIO11 renamed LED_AUX
- net LED_AUX: now also R23.1
- net GPIO6 renamed LED_PWR
- net LED_PWR: now also R21.1
- new net: D5.2 (A), R23.2
- new net: D2.2 (A), R21.2
- new net: D4.2 (A), R22.2
- new net +5V: C19.1, C22.1, D6.1 (K), FB1.2, R24.1
- new net 5V_EN: R26.1, U5.4 (EN)
- new net 5V_FB: R24.2, R25.1, U5.3 (FB)
- new net 5V_PRE: D6.2 (A), L1.2, U5.1 (SW)
- no-connect marks 13 -> 10
Other:
- note added: "(~4.96V)"
- note added: "3v3 Power"
- note added: "5v Power"
- note added: "Aux USB-A"
- note added: "LED"
- note added: "Level Shifter"
- note added: "Main Connector"
- note added: "SWD"
- note added: "Vout = 1.2 * (Rf + Rg) / Rg Rg <= 30k"
- note removed: "Power"
- note removed: "Power sources: - 5V from Main USB-C or External. Used as VBUS. Buck to 3v3. - 6V+ from VCC. Buck to 5v VBUS and 3v3."
- note removed: "gpio 16,17 and 20,21"
- moved on the sheet: C1, C10, C11, C12, C13, C14, C15, C16, C17, C22, C4, C5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

Commit message: new
Parts:
- removed C18: 4u7, Capacitor_SMD:C_0603_1608Metric, symbol Device:C_Small
- removed C19: 10u, Capacitor_SMD:C_0805_2012Metric, symbol Device:C_Small
- removed D1, D3: 1N5819WS, Diode_SMD:D_SOD-323, symbol Device:D_Schottky_Small
- removed D6: 40V/5A, Diode_SMD:D_SOD-323, symbol Device:D_Schottky_Small
- removed L1: 4u7, Inductor_SMD:L_1008_2520Metric, symbol Device:L_Small
- removed R24: 47k, Resistor_SMD:R_0603_1608Metric, symbol Device:R_Small
- removed R25: 15k, Resistor_SMD:R_0603_1608Metric, symbol Device:R_Small
- removed R26: 10k, Resistor_SMD:R_0402_1005Metric, symbol Device:R_Small_US
- removed U5: LGS6302, lcsc:SOT-23-5_L3.0-W1.6-P0.95-LS2.8-BL, symbol LCSC:LGS6302
- added J1: Conn_02x02_Odd_Even, Connector_PinHeader_2.54mm:PinHeader_2x02_P2.54mm_Vertical, symbol Connector_Generic:Conn_02x02_Odd_Even
Connections:
- net +5V is gone; now on net VBUS: C22.1, FB1.2
- net VCC is gone; now on net VBUS: C1.1, U3.3 (VI)
- net VBUS: now also J1.1 (Pin_1)
- net VCC_IN: now also J1.3 (Pin_3); no longer R13.1, R15.1, R17.1, R19.1
- new net VSH: J1.2 (Pin_2), J1.4 (Pin_4), R13.1, R15.1, R17.1, R19.1
Other:
- note removed: "(~4.96V)"
- note removed: "5v Power"
- note removed: "Vout = 1.2 * (Rf + Rg) / Rg Rg <= 30k"
