File: babelfish.kicad_sch (KiCad schematic)
At the start: 74 parts, among them J1 Conn_02x02_Odd_Even, J3 SWD, J5 IO_A, J7 USB_A, Q1 BSS138, SW1 K2-1836UQ-C3DW-06, U1 RP2040, U2 W25Q128JVS, U3 TPMCP1703T-5002E_CB, U4 GT-USB-7010ASV, U5 TPS2113ADRBR, U6 TPMCP1703T-3302E_CB, X1 X322512MSB4SI

Commit message: Power section done
Parts:
- removed SW1: K2-1836UQ-C3DW-06, lcsc:SW-SMD_4P-L2.8-W2.4-P1.60-LS3.0, symbol LCSC:K2-1836UQ-C3DW-06
- added SW1, SW2: TS342A2P-WZ, lcsc:SW-SMD_L4.0-W2.9-LS5.0, symbol LCSC:TS342A2P-WZ
- added SW3: SK12D07VG5_C3020419, lcsc:SW-TH_SHOU_SK12D07VG5, symbol LCSC:SK12D07VG5_C3020419
Connections:
- net GND: now also SW1.1, SW2.1, SW3.4, SW3.5
- net RUN: now also SW2.2
- net VCC_5V: now also SW3.3
- net VCC_IN: now also SW3.2; no longer C1.1, U3.3 (VIN)
- net ~{USB_BOOT}: now also SW1.2
- net U0_RX_C renamed GPIO17
- net U0_TX_C renamed GPIO16
- net U1_RX_C renamed GPIO21
- net U1_TX_C renamed GPIO20
- new net VCC_IN_SW: C1.1, SW3.1, U3.3 (VIN)
Other:
- note added: "5v0 Power (from VCC)"
- note added: "5v0 Power Mux"
- note added: "Can connect VCC_IN directly to VCC_5V, in case the host provides exactly 5V to avoid dropout."
- note removed: "5v0 Power"
- moved on the sheet: C10, C11, C12, C13, C14, C15, C16, C17, C18, C2, C20, C23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

Commit message: Added muxes
Parts:
- removed J5: IO_A, Connector_PinHeader_2.54mm:PinHeader_2x05_P2.54mm_Horizontal, symbol Connector_Generic:Conn_02x05_Odd_Even
- added C23, C24, C25, C26, C27: 100n, Capacitor_SMD:C_0402_1005Metric, symbol Device:C_Small
- added J3: DE9 Female, lcsc:DSUB-TH_DMR-9S, symbol Connector:DE9_Receptacle
- added U10, U7, U8, U9: 74HC4052PW,118, lcsc:TSSOP-16_L5.0-W4.4-P0.65-LS6.4-BL, symbol LCSC:74HC4052PW,118
- added U11: MAX3232IDR, lcsc:SOIC-16_L9.9-W3.9-P1.27-LS6.0-BL, symbol LCSC:MAX3232IDR
- added U12: AP2191WG-7, lcsc:SOT-25-5_L2.9-W1.6-P0.95-LS2.8-BL, symbol LCSC:AP2191WG-7
- C15: renamed from C18; value 0.1u -> 100n; footprint (none) -> Capacitor_SMD:C_0402_1005Metric
- C17: renamed from C23; footprint (none) -> Capacitor_SMD:C_0402_1005Metric
- C18: renamed from C20; value 0.1u -> 100n; footprint (none) -> Capacitor_SMD:C_0402_1005Metric
- C19: renamed from C1; footprint (none) -> Capacitor_SMD:C_0805_2012Metric; symbol Device:C_Polarized_Small -> Device:C_Small
- C20: renamed from C4; footprint (none) -> Capacitor_SMD:C_0805_2012Metric; symbol Device:C_Polarized_Small -> Device:C_Small
- C21: footprint (none) -> Capacitor_SMD:C_0805_2012Metric; symbol Device:C_Polarized_Small -> Device:C_Small
- C22: renamed from C19; footprint (none) -> Capacitor_SMD:C_0805_2012Metric; symbol Device:C_Polarized_Small -> Device:C_Small
- R2: renamed from R27; footprint (none) -> Resistor_SMD:R_0402_1005Metric
- R6: renamed from R24; footprint (none) -> Resistor_SMD:R_0402_1005Metric
- R8: renamed from R25; footprint (none) -> Resistor_SMD:R_0402_1005Metric
- R9: renamed from R26; footprint (none) -> Resistor_SMD:R_0402_1005Metric
- U5: renamed from U3; footprint lcsc.pretty:SOT-23-3_L2.9-W1.6-P1.90-LS2.8-BR -> lcsc:SOT-23-3_L2.9-W1.6-P1.90-LS2.8-BR
- U6: footprint lcsc.pretty:SOT-23-3_L2.9-W1.6-P1.90-LS2.8-BR -> lcsc:SOT-23-3_L2.9-W1.6-P1.90-LS2.8-BR
- renumbered C6 to C1, C16 to C10, C2 to C11, C3 to C12, C8 to C13, C10 to C14, C5 to C16, C7 to C2, C22 to C28, C17 to C3, C9 to C4, C11 to C5, C12 to C6, C13 to C7, C14 to C8, C15 to C9, D2 to D1, D4 to D2, D5 to D3, J3 to J2, J7 to J4, R20 to R1, R6 to R10, R1 to R11, R5 to R12, R11 to R13, R8 to R14, R21 to R15, R22 to R16, R23 to R17, R12 to R18, R13 to R19, R14 to R20, R15 to R21, R16 to R22, R17 to R23, R18 to R24, R19 to R25, R10 to R26, R9 to R27, R7 to R5, R2 to R7, U5 to U2, U4 to U3, U2 to U4
Connections:
- net U1_TX_CH is gone; now on net RX_B_2Y1: Q3.3 (D), R23.2
- net +3V3: now also C25.1, U10.16 (VCC), U11.16 (VCC), U7.16 (VCC), U8.16 (VCC), U9.16 (VCC)
- net 5V0: now also J1.1 (Pin_1), U12.5 (IN)
- net GND: now also C23.1, C25.2, C27.2, J3.1, U10.6 (~{E}), U10.7 (VEE), U10.8 (GND), U11.15 (GND), U12.2 (GND), U7.6 (~{E}), U7.7 (VEE), U7.8 (GND), U8.6 (~{E}), U8.7 (VEE), U8.8 (GND), U9.6 (~{E}), U9.7 (VEE), U9.8 (GND)
- net U0_RX_B: no longer Q2.2 (S), R20.2
- net U0_TX_B: no longer Q1.2 (S), R18.2
- net VBUS: no longer J1.1 (Pin_1)
- net VCC_IN: now also J3.6
- net U0_RX_A renamed RX_A
- net RX_A: now also U10.13 (1Z), U8.13 (1Z)
- net U0_RX_CH renamed RX_A_2Y1
- net RX_A_2Y1: now also U8.5 (2Y1)
- net U0_TX_A renamed TX_A
- net TX_A: now also U7.13 (1Z)
- net U0_TX_CH renamed TX_A_2Y1
- net TX_A_2Y1: now also U7.5 (2Y1)
- net U1_RX_B renamed RX_B_1Y1
- net RX_B_1Y1: now also U10.14 (1Y1); no longer U1.12 (GPIO9)
- net U1_RX_CH renamed RX_B_2Y1
- net RX_B_2Y1: now also U10.5 (2Y1)
- net U1_TX_B renamed TX_B_1Y1
- net TX_B_1Y1: now also U9.14 (1Y1); no longer U1.11 (GPIO8)
- net VSH renamed VSHIFT
- new net: C24.1, U11.1 (C1+)
- new net: C23.2, U11.2 (V+)
- new net: C24.2, U11.3 (C1-)
- new net: C26.1, U11.4 (C2+)
- new net: C26.2, U11.5 (C2-)
- new net: C27.1, U11.6 (V-)
- new net CH_A_S0: U7.10 (S0), U8.10 (S0)
- new net CH_A_S1: U7.9 (S1), U8.9 (S1)
- new net CH_B_S0: U10.10 (S0), U9.10 (S0)
- new net CH_B_S1: U10.9 (S1), U9.9 (S1)
- new net RX_A_1Y0: U8.12 (1Y0)
- new net RX_A_1Y1: Q2.2 (S), R20.2, U8.14 (1Y1)
- new net RX_A_1Y2: U11.12 (ROUT1), U8.15 (1Y2)
- new net RX_A_2Y0: U8.1 (2Y0)
- new net RX_A_2Y2: U11.13 (RIN1), U8.2 (2Y2)
- new net RX_A_CONN: J3.2, U8.3 (2Z)
- new net RX_B: U1.12 (GPIO9)
- new net RX_B_1Y0: U10.12 (1Y0)
- new net RX_B_1Y2: U10.15 (1Y2), U11.7 (DOUT2), U11.9 (ROUT2)
- new net RX_B_2Y0: U10.1 (2Y0)
- new net RX_B_2Y2: U10.2 (2Y2)
- new net RX_B_CONN: J3.7, U10.3 (2Z)
- new net TX_A_1Y0: U7.12 (1Y0)
- new net TX_A_1Y1: Q1.2 (S), R18.2, U7.14 (1Y1)
- new net TX_A_1Y2: U11.11 (DIN1), U7.15 (1Y2)
- new net TX_A_2Y0: U7.1 (2Y0)
- new net TX_A_2Y2: U11.14 (DOUT1), U7.2 (2Y2)
- new net TX_A_CONN: J3.3, U7.3 (2Z)
- new net TX_B: U1.11 (GPIO8), U9.13 (1Z)
- new net TX_B_1Y0: U9.12 (1Y0)
- new net TX_B_1Y2: U11.10 (DIN2), U9.15 (1Y2)
- new net TX_B_2Y0: U9.1 (2Y0)
- new net TX_B_2Y1: U9.5 (2Y1)
- new net TX_B_2Y2: U11.8 (RIN2), U9.2 (2Y2)
- new net TX_B_CONN: J3.8, U9.3 (2Z)
- new net USB2_EN: U12.4 (EN)
Other:
- note removed: "Main Connector"
- moved on the sheet: C15, C17, C18, C28, FB1, J2, J4, R10, R2, R26, R27, R5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

Commit message: Layout v2 done
Parts:
- removed FB1: FerriteBead_Small, Inductor_SMD:L_0805_2012Metric, symbol Device:FerriteBead_Small
- removed J1: Conn_02x02_Odd_Even, Connector_PinHeader_2.54mm:PinHeader_2x02_P2.54mm_Vertical, symbol Connector_Generic:Conn_02x02_Odd_Even
- added C29, C31: 10u, Capacitor_SMD:C_0805_2012Metric, symbol Device:C_Small
- added C30: 100n, Capacitor_SMD:C_0402_1005Metric, symbol Device:C_Small
- added J1: Shifter Power, Connector_PinHeader_2.54mm:PinHeader_1x03_P2.54mm_Vertical, symbol Connector_Generic:Conn_01x03
- added R28: 10k, Resistor_SMD:R_0402_1005Metric, symbol Device:R_Small
- C28: value 10u -> 100n; footprint Capacitor_SMD:C_0805_2012Metric -> Capacitor_SMD:C_0402_1005Metric
Connections:
- net GPIO2 is gone; now on net CH_A_S0: U1.4 (GPIO2)
- net GPIO20 is gone; now on net USB2_EN: U1.31 (GPIO20)
- net GPIO21 is gone; now on net USB2_FLG: U1.32 (GPIO21)
- net GPIO23 is gone; now on net STAT_5V0: U1.35 (GPIO23)
- net GPIO3 is gone; now on net CH_A_S1: U1.5 (GPIO3)
- net RX_A_2Y0 is gone; now on net RX_A_Y0_THRU: U8.1 (2Y0)
- net RX_B_2Y0 is gone; now on net RX_B_Y0_THRU: U10.1 (2Y0)
- net TX_A_2Y0 is gone; now on net TX_A_Y0_THRU: U7.1 (2Y0)
- net TX_B_2Y0 is gone; now on net TX_B_Y0_THRU: U9.1 (2Y0)
- net U0_RX_B is gone; now on net GPIO13: U1.16 (GPIO13)
- net U0_TX_B is gone; now on net GPIO12: U1.15 (GPIO12)
- net +3V3: now also R28.2
- net 5V0: now also C30.1, C31.1, J1.3 (Pin_3)
- net GND: now also C29.2, C30.2, C31.2
- net GPIO14: now also J3.4
- net RX_A: no longer U10.13 (1Z)
- net RX_A_1Y1: now also Q1.2 (S), R18.2; no longer Q2.2 (S), R20.2
- net RX_A_2Y1: now also Q1.3 (D), R19.2; no longer Q2.3 (D), R21.2
- net RX_A_CONN: now also J3.7; no longer J3.2
- net RX_B: now also U10.13 (1Z)
- net RX_B_1Y2: no longer U11.7 (DOUT2)
- net RX_B_2Y1: no longer Q3.3 (D), R23.2
- net RX_B_2Y2: now also U11.8 (RIN2)
- net RX_B_CONN: now also J3.8; no longer J3.7
- net TX_A_1Y1: now also Q2.2 (S), R20.2; no longer Q1.2 (S), R18.2
- net TX_A_2Y1: now also Q2.3 (D), R21.2; no longer Q1.3 (D), R19.2
- net TX_A_CONN: now also J3.2; no longer J3.3
- net TX_B_2Y1: now also Q3.3 (D), R23.2
- net TX_B_2Y2: now also U11.7 (DOUT2); no longer U11.8 (RIN2)
- net TX_B_CONN: now also J3.3; no longer J3.8
- net VBUS: no longer C28.1
- net VCC_IN: now also J1.1 (Pin_1)
- net VSHIFT: now also J1.2 (Pin_2)
- net PWR_VSNS: now reaches R6.2, R8.1, U2.3 (VSNS)
- net VBUS_OUT: now reaches J4.1 (VBUS)
- net VBUS_OUT: now also C28.1, U12.1 (OUT), C29.1
- net USB2_FLG: now reaches U12.3 (FLG)
- net USB2_FLG: now also R28.1
- net GPIO13: now reaches J3.5
- net GPIO12: now reaches J3.9
- net RX_A_1Y0 renamed RX_A_Y0_THRU
- net RX_B_1Y0 renamed RX_B_Y0_THRU
- net TX_A_1Y0 renamed TX_A_Y0_THRU
- net TX_B_1Y0 renamed TX_B_Y0_THRU
- no-connect marks 10 -> 15
Other:
- note added: "NB: this cap near pin 44"
- note added: "Signal Mux/Demux"
- note removed: "NB: C10 near pin 44"
- moved on the sheet: U12

Commit message: V2 export WIP
Connections:
- net +3V3: now also J3.9
- net GPIO12: no longer J3.9
Changed lines of the file:
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@@
+    (stroke (width 0) (type default))
+  )
+  (wire (pts (xy 156.845 203.2) (xy 149.225 203.2))
     (stroke (width 0) (type default))
   )
@@
     (stroke (width 0) (type default))
   )
+  (wire (pts (xy 156.845 196.215) (xy 156.845 203.2))
+    (stroke (width 0) (type default))
+  )
   (wire (pts (xy 40.005 227.965) (xy 43.18 227.965))
     (stroke (width 0) (type default))
@@
   )
   (wire (pts (xy 20.955 151.13) (xy 33.655 151.13))
-    (stroke (width 0) (type default))
-  )
-  (wire (pts (xy 149.225 203.2) (xy 161.925 203.2))
     (stroke (width 0) (type default))
   )
@@
   (label "RX_B_2Y2" (at 43.18 240.665 0) (fields_autoplaced)
     (effects (font (size 1.27 1.27)) (justify left bottom))
-  )
-  (label "GPIO12" (at 161.925 203.2 180) (fields_autoplaced)
-    (effects (font (size 1.27 1.27)) (justify right bottom))
   )
   (label "VSHIFT" (at 344.805 161.29 0) (fields_autoplaced)
@@
         )
       )
+    )
+  )
+  (symbol (lib_id "power:+3V3") (at 156.845 196.215 0) (unit 1)
+    (in_bom yes) (on_board yes) (dnp no) (fields_autoplaced)
+    (property "Reference" "#PWR061" (at 156.845 200.025 0)
+      (effects (font (size 1.27 1.27)) hide)
+    )
+    (property "Value" "+3V3" (at 156.845 191.135 0)
+      (effects (font (size 1.27 1.27)))
+    )
+    (property "Footprint" "" (at 156.845 196.215 0)
+      (effects (font (size 1.27 1.27)) hide)
+    )
+    (property "Datasheet" "" (at 156.845 196.215 0)
+      (effects (font (size 1.27 1.27)) hide)
+    )
+    (pin "1")
+    (instances
+      (project "babelfish"
+        (path "/25a7582e-3999-4fda-9acd-cd1e305548b6"
+          (reference "#PWR061") (unit 1)
+        )
+      )

Commit message: v2
Parts:
- D3: value Blue -> Red
- R15, R16, R17: value 68 -> 1k
Changed lines of the file:
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@@
   (symbol (lib_id "Device:LED_Small") (at 45.085 171.45 180) (unit 1)
     (in_bom yes) (on_board yes) (dnp no) (fields_autoplaced)
-    (property "Reference" "D3" (at 45.0215 166.37 0)
-      (effects (font (size 1.27 1.27)))
-    )
-    (property "Value" "Blue" (at 45.0215 168.91 0)
+    (property "Reference" "D3" (at 45.0215 165.1 0)
+      (effects (font (size 1.27 1.27)))
+    )
+    (property "Value" "Red" (at 45.0215 167.64 0)
       (effects (font (size 1.27 1.27)))
     )
@@
       (effects (font (size 1.27 1.27)))
     )
-    (property "Value" "68" (at 36.195 148.59 90)
+    (property "Value" "1k" (at 36.195 148.59 90)
       (effects (font (size 1.27 1.27)))
     )
@@
       (effects (font (size 1.27 1.27)))
     )
-    (property "Value" "68" (at 36.195 158.75 90)
+    (property "Value" "1k" (at 36.195 158.75 90)
       (effects (font (size 1.27 1.27)))
     )
@@
       (effects (font (size 1.27 1.27)))
     )
-    (property "Value" "68" (at 36.195 168.91 90)
-      (effects (font (size 1.27 1.27)))
-    )
+    (property "Value" "1k" (at 36.195 168.91 90)
+      (effects (font (size 1.27 1.27)))
+    )
