File: saved_stack_usb.kicad_sch (KiCad schematic)
At the start: 59 parts, among them J3 SWD, J4 Shifter Power, J5 IO_A, J7 USB_A, Q1 BSS138, SW1 K2-1156SP-D5SW-05, U1 NCP1117-3.3_SOT223, U2 W25Q128JVS, U3 RP2040, U4 GT-USB-7010ASV, X1 X322512MSB4SI

Commit message: rev 0.1
Parts:
- removed SW1: K2-1156SP-D5SW-05, lcsc:SW-SMD_4P-L6.3-W6.2-P4.00-LS9.4-TL, symbol LCSC:K2-1156SP-D5SW-05
- removed U4: GT-USB-7010ASV, lcsc:USB-C-SMD_G-SWITCH_GT-USB-7010ASV, symbol LCSC:GT-USB-7010ASV
- added C18, C19, C20, C21: 0.1uf, Capacitor_SMD:C_0402_1005Metric, symbol Device:C_Polarized_Small_US
- added C23, C24: 30p, Capacitor_SMD:C_0402_1005Metric, symbol Device:C
- added D2: 1N5819WS, Diode_SMD:D_SOD-323, symbol Device:D_Schottky_Small
- added J1: TYPE-C-31-M-12, Connector_USB:USB_C_Receptacle_HRO_TYPE-C-31-M-12, symbol Connector:USB_C_Receptacle_USB2.0
- added J2: Conn_01x02, Connector_PinHeader_2.54mm:PinHeader_1x02_P2.54mm_Vertical, symbol Connector_Generic:Conn_01x02
- added J6: IO_B, Connector_PinHeader_2.54mm:PinHeader_2x05_P2.54mm_Horizontal, symbol Connector_Generic:Conn_02x05_Odd_Even
- added R21: 1k, symbol Device:R_Small
- added U4: WS3232ECY, Package_SO:TSSOP-16_4.4x5mm_P0.65mm, symbol dk_Interface-Drivers-Receivers-Transceivers:MAX3232CPE_
- added U5: FE1_1S, lcsc:SSOP-28_L9.9-W3.9-P0.64-LS6.0-BL-1, symbol LCSC:FE1_1S
- added USB1: Double_layer_DIP_90°_black, lcsc:USB-A-TH_USB-M-51, symbol LCSC:Double_layer_DIP_90°_black
- added X2: X322512MSB4SI, lcsc:OSC-SMD_4P-L3.2-W2.5-BL, symbol LCSC:X322512MSB4SI
- R1, R10, R11, R2, R3, R4, R5, R9: footprint Resistor_SMD:R_0402_1005Metric -> Capacitor_SMD:C_0402_1005Metric
- R20: footprint Resistor_SMD:R_0402_1005Metric -> (none)
Connections:
- net +3V3: now also C20.2, U4.16 (VCC)
- net GND: now also R6.1, R7.1, C21.1, J1.A1 (GND), J1.A12 (GND), J1.A8 (SBU1), J1.B1 (GND), J1.B12 (GND), J1.B8 (SBU2), J1.S1 (SHIELD), J2.2 (Pin_2), J6.10 (Pin_10), U4.15 (GND), X2.2 (GND), X2.4 (GND); no longer R6.2, R7.2
- net GPIO26: now also J6.2 (Pin_2)
- net GPIO27: now also J6.4 (Pin_4)
- net GPIO28: now also J6.6 (Pin_6)
- net GPIO29: now also J6.8 (Pin_8)
- net SH_REF: no longer J4.1 (Pin_1), J4.3 (Pin_3), J4.5 (Pin_5)
- net U0_RX_B: now also U4.12 (R2OUT); no longer Q2.2 (S), R14.2
- net U0_RX_C: now also Q2.2 (S), R14.2
- net U0_TX_B: now also U4.11 (T2IN); no longer Q1.2 (S), R12.2
- net U0_TX_C: now also Q1.2 (S), R12.2
- net U1_RX_B: now also U4.9 (R1OUT); no longer Q4.2 (S), R18.2
- net U1_RX_C: now also Q4.2 (S), R18.2
- net U1_TX_B: now also U4.10 (T1IN); no longer Q3.2 (S), R16.2
- net U1_TX_C: now also Q3.2 (S), R16.2
- net USB_D+: now also J1.A6 (D+), J1.B6 (D+)
- net USB_D-: now also J1.A7 (D-), J1.B7 (D-)
- net VBUS: now also J1.A4 (VBUS), J1.A9 (VBUS), J1.B4 (VBUS), J1.B9 (VBUS)
- net VCC: now also D2.1 (K)
- net ~{USB_BOOT}: now also J2.1 (Pin_1)
- new net: J1.A5 (CC1), R6.2
- new net: J1.B5 (CC2), R7.2
- new net: J4.1 (Pin_1), J4.3 (Pin_3), J4.5 (Pin_5)
- new net: C23.1, X2.1 (OSC1)
- new net: C24.1, X2.3 (OSC2)
- new net: C24.2, U5.3 (XIN)
- new net: C18.1, U4.1 (C1+)
- new net: C20.1, U4.2 (V+)
- new net: C18.2, U4.3 (C1-)
- new net: C19.1, U4.4 (C2+)
- new net: C19.2, U4.5 (C2-)
- new net: C21.2, U4.6 (V-)
- new net: C23.2, R21.1
- new net: R21.2, U5.2 (XOUT)
- new net U0_232_RX: J6.7 (Pin_7), U4.13 (R2IN)
- new net U0_232_TX: J6.5 (Pin_5), U4.14 (T2OUT)
- new net U1_232_RX: J6.3 (Pin_3), U4.8 (R1IN)
- new net U1_232_TX: J6.1 (Pin_1), U4.7 (T1OUT)
- new net VCC2_IN: D2.2 (A), J6.9 (Pin_9)
- no-connect marks 13 -> 9
Other:
- note added: "USB2 USB-A Host"
- moved on the sheet: R6, R7
