File: babelfish.kicad_pcb (KiCad board)
At the start: 4 copper layers, 56 x 45.2 mm, 97 parts, among them J1 Shifter Power, J2 SWD, J3 DE9 Female, J4 USB_A, Q1 BSS138, SW1 TS342A2P-WZ, SW2 TS342A2P-WZ, SW3 SK12D07VG5_C3020419, U1 RP2040, U10 74HC4052PW,118, U11 MAX3232IDR, U12 AP2191WG-7, U2 TPS2113ADRBR, U3 GT-USB-7010ASV, U4 W25Q128JVS, U5 TPMCP1703T-5002E_CB, U6 TPMCP1703T-3302E_CB, U7 74HC4052PW,118, U8 74HC4052PW,118, U9 74HC4052PW,118, X1 X322512MSB4SI

Commit message: v2
Changed lines of the file:
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@@
       (psnegative false)
       (psa4output false)
-      (plotreference true)
+      (plotreference false)
       (plotvalue false)
       (plotinvisibletext false)
@@
       (drillshape 0)
       (scaleselection 1)
-      (outputdirectory "gerbers")
+      (outputdirectory "v2")
     )
   )
@@
   (segment (start 117.9105 91.1226) (end 119.0196 92.2317) (width 0.286) (layer "F.Cu") (net 19))
   (segment (start 115.463 91.1265) (end 116.8866 91.1265) (width 0.15) (layer "F.Cu") (net 21))
-  (segment (start 116.0243 92.0878) (end 116.8905 92.0878) (width 0.15) (layer "F.Cu") (net 22))
-  (segment (start 115.463 91.5265) (end 116.0243 92.0878) (width 0.15) (layer "F.Cu") (net 22))
+  (segment (start 116.5878 92.0878) (end 116.8905 92.0878) (width 0.15) (layer "F.Cu") (net 22))
+  (segment (start 115.463 91.5265) (end 116.0265 91.5265) (width 0.15) (layer "F.Cu") (net 22))
+  (segment (start 116.0265 91.5265) (end 116.5878 92.0878) (width 0.15) (layer "F.Cu") (net 22))
   (segment (start 116.2 93.5135) (end 116.2 93.8) (width 0.15) (layer "F.Cu") (net 23))
   (segment (start 113.8255 92.364) (end 113.8255 92.790409) (width 0.15) (layer "F.Cu") (net 23))
