File: hardware/babelfish.kicad_pcb (KiCad board)
At the start: 4 copper layers, 76 x 45.2 mm, 103 parts, among them J2 SWD, J3 DE9 Female, J4 USB_A, Q1 BSS138, SW1 TS342A2P-WZ, SW2 TS342A2P-WZ, U1 RP2040, U11 MAX3232IDR, U12 AP2191WG-7, U2 TPS2113ADRBR, U3 GT-USB-7010ASV, U36 TPS62933, U4 W25Q128JVS, U6 TPMCP1703T-3302E_CB, U7 74HC4052PW,118, U8 74HC4052PW,118, X1 X322512MSB4SI

Commit message: v3 rc0
Parts:
- removed C38: 100n, Capacitor_SMD:C_0402_1005Metric
- removed C39: 33n, Capacitor_SMD:C_01005_0402Metric
- removed C40: 47p, Capacitor_SMD:C_0402_1005Metric
- removed C41: 22u, Capacitor_SMD:C_0805_2012Metric
- removed DIP2: DSWB04LHGET, lcsc:SW-TH_DSWB04LHGET
- removed L36: 2.7uH, lcsc:IND-SMD_L6.0-W6.0_FNR60XXS
- removed R36: 52k3, Resistor_SMD:R_0402_1005Metric
- removed R37: 15k, Resistor_SMD:R_0402_1005Metric
- removed R38: 10k, Resistor_SMD:R_0402_1005Metric
- removed U36: TPS62933, Package_TO_SOT_SMD:SOT-583-8
- added RAc: TestPoint, TestPoint:TestPoint_Pad_D2.0mm, B.Cu at (70.0, 63.0)
- added RBc: TestPoint, TestPoint:TestPoint_Pad_D2.0mm, B.Cu at (65.0, 58.0)
- added RX_A: TestPoint, TestPoint:TestPoint_Pad_D2.0mm, B.Cu at (52.8, 50.6)
- added RX_B: TestPoint, TestPoint:TestPoint_Pad_D2.0mm, B.Cu at (47.8, 44.2)
- added TAc: TestPoint, TestPoint:TestPoint_Pad_D2.0mm, B.Cu at (65.0, 63.0)
- added TBc: TestPoint, TestPoint:TestPoint_Pad_D2.0mm, B.Cu at (70.0, 58.0)
- added TX_A: TestPoint, TestPoint:TestPoint_Pad_D2.0mm, B.Cu at (38.5, 36.6)
- added TX_B: TestPoint, TestPoint:TestPoint_Pad_D2.0mm, B.Cu at (50.8, 48.2)
- 3V3: renamed from TP1; footprint TestPoint:TestPoint_Pad_D1.0mm -> TestPoint:TestPoint_Pad_D2.0mm; moved to B.Cu
- 5V0: renamed from TP4; footprint TestPoint:TestPoint_Pad_D1.0mm -> TestPoint:TestPoint_Pad_D2.0mm; moved to B.Cu
- C36: footprint Capacitor_SMD:C_01005_0402Metric -> Capacitor_SMD:C_0402_1005Metric
- C37: value 10u -> 100n; footprint Capacitor_SMD:C_0805_2012Metric -> Capacitor_SMD:C_0402_1005Metric
- GND: renamed from TP5; footprint TestPoint:TestPoint_Pad_D1.0mm -> TestPoint:TestPoint_Pad_D2.0mm; moved to B.Cu
- U7, U8: value 74HC4052PW,118 -> SN74CBT3253CPWR; footprint lcsc:TSSOP-16_L5.0-W4.4-P0.65-LS6.4-BL -> lcsc:TSSOP-16_L5.0-W4.4-P0.65-LS6.4-TL
- VBUS: renamed from TP3; footprint TestPoint:TestPoint_Pad_D1.0mm -> TestPoint:TestPoint_Pad_D2.0mm; moved to B.Cu
- VCC_5V: renamed from TP2; footprint TestPoint:TestPoint_Pad_D1.0mm -> TestPoint:TestPoint_Pad_D2.0mm; moved to B.Cu
- moved VCC_5V 71.3 mm to (89.1, 40.2), turned to 180 degrees
- moved VBUS 66.5 mm to (78.3, 41.5), turned to 180 degrees
- moved 3V3 63.1 mm to (85.5, 51.6), turned to 180 degrees
- moved kibuzzard-644F3679 57.4 mm to (82.0, 63.5)
- moved 5V0 56.3 mm to (69.1, 45.0), turned to 180 degrees
- moved J2 48.9 mm to (74.4, 26.7), turned to 0 degrees
- moved C36 33.0 mm to (43.7, 32.5), turned to 90 degrees
- moved C37 28.4 mm to (43.7, 41.5), turned to 90 degrees
- moved H3 21.7 mm to (90.0, 26.0)
- moved kibuzzard-644F39EB 18.8 mm to (27.4, 32.7)
- moved GND 9.02 mm to (89.1, 33.6), turned to 180 degrees
- moved R2 7.88 mm to (76.6, 38.9), turned to 0 degrees
- moved J4 6.66 mm to (68.4, 54.2)
- moved R26 6.66 mm to (67.3, 50.9)
- moved R27 6.66 mm to (69.5, 50.9)
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Connections:
- net /RX_A_1Y1 renamed /RX_A_SHIFTER
- net /RX_A_2Y1 renamed /RX_A_SHIFTER_OUT
- net /RX_A_2Y2 renamed /RX_A_MAX_OUT
- net /RX_B_1Y1 renamed /RX_B_SHIFTER
- net /RX_B_2Y1 renamed /RX_B_SHIFTER_OUT
- net /RX_B_2Y2 renamed /RX_B_MAX_OUT
- net /TX_A_2Y1 renamed /TX_A_SHIFTER_OUT
- net /TX_A_2Y2 renamed /TX_A_MAX_OUT
- net /TX_B_2Y1 renamed /TX_B_SHIFTER_OUT
- net /TX_B_2Y2 renamed /TX_B_MAX_OUT
- C36 pad 1: Net-(U36-SW) -> GND
- C36 pad 2: Net-(U36-BST) -> /5V0
- C37 pad 1: /VCC_IN_SW -> GND
- C37 pad 2: GND -> /5V0
- J3 pad 4: /GPIO15 -> /GPIO14
- J3 pad 5: /GPIO14 -> /GPIO15
- J3 pad 6: /VCC_IN -> /VCC_5V
- Q2 pad 2: /TX_A_1Y1 -> /TX_A_SHIFTER
- Q3 pad 2: /TX_B_1Y1 -> /TX_B_SHIFTER
- R19 pad 1: /VSHIFT -> /5V0
- R20 pad 2: /TX_A_1Y1 -> /TX_A_SHIFTER
- R21 pad 1: /VSHIFT -> /5V0
- R22 pad 2: /TX_B_1Y1 -> /TX_B_SHIFTER
- R23 pad 1: /VSHIFT -> /5V0
- R25 pad 1: /VSHIFT -> /5V0
- U11 pad 10: /TX_B_1Y2 -> /TX_B_MAX
- U11 pad 11: /TX_A_1Y2 -> /TX_A_MAX
- U11 pad 12: /RX_A_1Y2 -> /RX_A_MAX
- U11 pad 9: /RX_B_1Y2 -> /RX_B_MAX
- U7 pad 1: /RX_A_CONN -> GND
- U7 pad 10: /CH_A_S0 -> /TX_A_CONN
- U7 pad 11: unconnected-(U7-1Y3-Pad11) -> /TX_A_SHIFTER
- U7 pad 12: /TX_A_CONN -> /TX_A_MAX
- U7 pad 13: /TX_A -> unconnected-(U7-2B4-Pad13)
- U7 pad 14: /TX_A_1Y1 -> /CH_A_S0
- U7 pad 15: /TX_A_1Y2 -> GND
- U7 pad 16: +3V3 -> /5V0
- U7 pad 2: /RX_A_1Y2 -> /CH_A_S1
- U7 pad 3: /RX_A -> unconnected-(U7-1B4-Pad3)
- U7 pad 4: unconnected-(U7-2Y3-Pad4) -> /RX_A_MAX
- U7 pad 6: GND -> /RX_A_CONN
- U7 pad 7: GND -> /RX_A
- U7 pad 9: /CH_A_S1 -> /TX_A
- U8 pad 1: /RX_B_CONN -> GND
- U8 pad 10: /CH_B_S0 -> /TX_B_CONN
- U8 pad 11: unconnected-(U8-1Y3-Pad11) -> /TX_B_SHIFTER
- U8 pad 12: /TX_B_CONN -> /TX_B_MAX
- U8 pad 13: /TX_B -> unconnected-(U8-2B4-Pad13)
- U8 pad 14: /TX_B_1Y1 -> /CH_B_S0
- U8 pad 15: /TX_B_1Y2 -> GND
- U8 pad 16: +3V3 -> /5V0
- U8 pad 2: /RX_B_1Y2 -> /CH_B_S1
- U8 pad 3: /RX_B -> unconnected-(U8-1B4-Pad3)
- U8 pad 4: unconnected-(U8-2Y3-Pad4) -> /RX_B_MAX
- U8 pad 6: GND -> /RX_B_CONN
- U8 pad 7: GND -> /RX_B
- U8 pad 9: /CH_B_S1 -> /TX_B
- VCC_5V pad 1: /VCC_IN -> /VCC_5V
Routing:
- net /5V0: track 6.56 -> 89.0 mm, vias 0 -> 6
- net /TX_A_SHIFTER_OUT: track 1.52 -> 50.0 mm, vias 0 -> 1
- net /RX_B_SHIFTER_OUT: track 1.52 -> 49.1 mm, vias 0 -> 1
- net /RX_A_SHIFTER_OUT: track 1.55 -> 46.6 mm, vias 0 -> 1
- net /VCC_IN: track 43.8 -> 0.00 mm
- net /VCC_IN_SW: track 43.0 -> 0.00 mm, vias 2 -> 0
- net /RX_A_CONN: track 63.1 -> 104.9 mm, vias 0 -> 2
- net /TX_A_CONN: track 65.1 -> 103.9 mm, vias 0 -> 5
- net /GPIO14: track 0.00 -> 33.3 mm, vias 0 -> 2
- net /TX_B_SHIFTER_OUT: track 1.47 -> 34.8 mm, vias 0 -> 1
- net /RUN: track 3.69 -> 36.9 mm, vias 0 -> 2
- net /LED_PWR: track 0.00 -> 32.4 mm, vias 0 -> 4
- net /GPIO15: track 0.00 -> 31.6 mm, vias 0 -> 2
- net /LED_P_OK: track 0.00 -> 29.5 mm, vias 0 -> 2
- net /SWD: track 0.00 -> 29.4 mm, vias 0 -> 2
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- removed copper zone on F.Cu, net /VCC_5V
- removed copper zone on F.Cu, net /VCC_IN_SW
- removed copper zone on F.Cu, net Net-(U36-FB)
- removed copper zone on F.Cu, net Net-(U36-SW)
Other:
- board size 76 x 45.2 mm -> 72 x 43.4 mm
- board text added: "232"
- board text added: "5V"
- board text added: "RX_A"
- board text added: "RX_B"
- board text added: "TX_A"
- board text added: "TX_B"
- board text added: "off= 3V3"
- board text removed: "3"
- board text removed: "5"
- board text removed: "G"
- board text removed: "POWER CFG"
- board text removed: "S"
- board text removed: "V"
