File: hardware/babelfish.kicad_pcb (KiCad board)
At the start: 4 copper layers, 72 x 43.4 mm, 101 parts, among them J2 SWD, J3 DE9 Female, J4 USB_A, Q1 BSS138, SW1 TS342A2P-WZ, SW2 TS342A2P-WZ, U1 RP2040, U11 MAX3232IDR, U12 AP2191WG-7, U2 TPS2113ADRBR, U3 GT-USB-7010ASV, U4 W25Q128JVS, U6 TPMCP1703T-3302E_CB, U7 SN74CBT3253CPWR, U8 SN74CBT3253CPWR, X1 X322512MSB4SI

Commit message: v3 rc2
Routing:
- net +1V1: track 18.9 -> 29.1 mm, vias 0 -> 2
- net /RUN: track 36.9 -> 38.4 mm
- net GND: track 96.3 -> 96.9 mm
Changed lines of the file:
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@@
 		(sheetname "Root")
 		(sheetfile "babelfish.kicad_sch")
-		(attr exclude_from_pos_files)
+		(attr exclude_from_pos_files exclude_from_bom)
 		(fp_circle
 			(center 0 0)
@@
 		(sheetname "Root")
 		(sheetfile "babelfish.kicad_sch")
-		(attr through_hole)
+		(attr through_hole exclude_from_pos_files exclude_from_bom)
 		(fp_circle
 			(center 3.2 -2.2)
@@
 		(sheetname "Root")
 		(sheetfile "babelfish.kicad_sch")
-		(attr exclude_from_pos_files)
+		(attr exclude_from_pos_files exclude_from_bom)
 		(fp_circle
 			(center 0 0)
@@
 		(sheetname "Root")
 		(sheetfile "babelfish.kicad_sch")
-		(attr smd)
+		(attr smd exclude_from_pos_files exclude_from_bom)
 		(fp_line
 			(start -0.153641 0.38)
@@
 		(sheetname "Root")
 		(sheetfile "babelfish.kicad_sch")
-		(attr exclude_from_pos_files)
+		(attr exclude_from_pos_files exclude_from_bom)
 		(fp_circle
 			(center 0 0)
@@
 		(sheetname "Root")
 		(sheetfile "babelfish.kicad_sch")
-		(attr exclude_from_pos_files)
+		(attr exclude_from_pos_files exclude_from_bom)
 		(fp_circle
 			(center 0 0)
@@
 		(sheetname "Root")
 		(sheetfile "babelfish.kicad_sch")
-		(attr exclude_from_pos_files)
+		(attr exclude_from_pos_files exclude_from_bom)
 		(fp_circle
 			(center 0 0)
@@
 		(sheetname "Root")
 		(sheetfile "babelfish.kicad_sch")
-		(attr exclude_from_pos_files)
+		(attr exclude_from_pos_files exclude_from_bom)
 		(fp_circle
 			(center 0 0)
@@
 		(sheetname "Root")
 		(sheetfile "babelfish.kicad_sch")
-		(attr exclude_from_pos_files)
+		(attr exclude_from_pos_files exclude_from_bom)
 		(fp_circle
 			(center 0 0)
@@
 	)
 	(segment
-		(start 56.625 34.15)
-		(end 56.6255 34.1495)
-		(width 0.2)
-		(layer "F.Cu")
-		(net 1)
-	)
-	(segment
 		(start 24.1 47.72883)
 		(end 25.02883 47.72883)
@@
 	)
 	(segment
+		(start 58.2 34.2)
+		(end 57.5755 34.8245)
+		(width 0.2)
+		(layer "F.Cu")
+		(net 1)
+	)
+	(segment
 		(start 36.9 46.668086)
 		(end 36.9 46.8)
@@
 	)
 	(segment
+		(start 58.2 34.125)
+		(end 58.2 34.2)
+		(width 0.2)
+		(layer "F.Cu")
+		(net 1)
+	)
+	(segment
 		(start 26.679985 48.1)
 		(end 26.679985 46.32883)
@@
 	)
 	(segment
-		(start 57.5755 34.1755)
-		(end 57.575 34.175)
-		(width 0.2)
-		(layer "F.Cu")
-		(net 1)
-	)
-	(segment
 		(start 75.08 38.78)
 		(end 75.1 38.8)
@@
 	)
 	(segment
-		(start 56.6255 34.1505)
-		(end 56.625 34.15)
-		(width 0.2)
-		(layer "F.Cu")
-		(net 1)
-	)
-	(segment
 		(start 42.9 23.6)
 		(end 42.9 24.8)
@@
 	)
 	(segment
-		(start 56.6255 34.1495)
-		(end 56.6255 34.1255)
-		(width 0.2)
-		(layer "F.Cu")
-		(net 1)
-	)
-	(segment
 		(start 56.7255 46.45)
 		(end 56.7255 45.464)
@@
 	)
 	(segment
-		(start 56.6255 35.039)
-		(end 56.6255 34.1505)
-		(width 0.2)
-		(layer "F.Cu")
-		(net 1)
-	)
-	(segment
 		(start 42.9 28.05)
 		(end 42.9 29.5)
@@
 	)
 	(segment
+		(start 57.5755 34.8245)
+		(end 57.5755 35.04)
+		(width 0.2)
+		(layer "F.Cu")
+		(net 1)
+	)
+	(segment
 		(start 25.02883 47.72883)
 		(end 25.6 48.3)
@@
 	)
 	(segment
-		(start 57.575 34.175)
-		(end 57.575 34.125)
+		(start 56.6255 35.039)
+		(end 56.6255 34.8745)
 		(width 0.2)
 		(layer "F.Cu")
@@
 	)
 	(segment
+		(start 56.6255 34.8745)
+		(end 57.4 34.1)
+		(width 0.2)
+		(layer "F.Cu")
+		(net 1)
+	)
+	(segment
 		(start 36.109728 36.977814)
 		(end 34.3 37)
@@
 	)
 	(segment
-		(start 57.5755 35.04)
-		(end 57.5755 34.1755)
-		(width 0.2)
-		(layer "F.Cu")
-		(net 1)
-	)
-	(segment
 		(start 73.2 34.65)
 		(end 73.219949 34.669949)
@@
 	)
 	(via
-		(at 57.575 34.125)
+		(at 58.2 34.125)
 		(size 0.6)
 		(drill 0.35)
@@
 	)
 	(via
-		(at 56.625 34.125)
+		(at 57.4 34.1)
 		(size 0.6)
 		(drill 0.35)
@@
 	)
 	(segment
+		(start 56.6255 35.999)
+		(end 56.3265 35.7)
+		(width 0.15)
+		(layer "F.Cu")
+		(net 6)
+	)
+	(segment
 		(start 57.8 39.8)
 		(end 59.4 39.8)
@@
 	)
 	(segment
+		(start 60.97 37.33)
+		(end 60.4055 37.33)
+		(width 0.2)
+		(layer "F.Cu")
+		(net 6)
+	)
+	(segment
+		(start 61.3 37)
+		(end 60.97 37.33)
+		(width 0.2)
+		(layer "F.Cu")
+		(net 6)
+	)
+	(segment
 		(start 59.9 43.5)
 		(end 59.4 44)
@@
 	)
 	(segment
-		(start 56.6255 36.689)
-		(end 56.6358 36.6787)
-		(width 0.2)
+		(start 60.78825 46.81175)
+		(end 60.6155 46.639)
+		(width 0.15)
 		(layer "F.Cu")
 		(net 6)
 	)
 	(segment
-		(start 60.78825 46.81175)
-		(end 60.6155 46.639)
+		(start 56.5 34.1)
+		(end 56.4 34.1)
 		(width 0.15)
 		(layer "F.Cu")
@@
 	)
 	(segment
+		(start 56.3265 35.7)
+		(end 55.9 35.2735)
+		(width 0.15)
+		(layer "F.Cu")
+		(net 6)
+	)
+	(segment
 		(start 57.5255 38.589)
 		(end 57.5255 37.865496)
@@
 		(start 56.6358 36.6787)
 		(end 56.6358 36.0093)
-		(width 0.2)
+		(width 0.15)
 		(layer "F.Cu")
 		(net 6)
@@
 	)
 	(segment
+		(start 55.9 35.2735)
+		(end 55.9 34.9)
+		(width 0.15)
+		(layer "F.Cu")
+		(net 6)
+	)
+	(segment
 		(start 60.252024 37.33)
 		(end 60.4055 37.33)
@@
 	)
 	(segment
+		(start 55.9 34.9)
+		(end 55.9 34.6)
+		(width 0.15)
+		(layer "F.Cu")
+		(net 6)
+	)
+	(segment
 		(start 58.3255 45.464)
 		(end 58.3255 46.239)
@@
 	)
 	(segment
-		(start 56.6358 36.6993)
-		(end 56.6255 36.689)
+		(start 55.9 34.6)
+		(end 56.5 34.1)
 		(width 0.15)
 		(layer "F.Cu")
@@
 	)
 	(segment
+		(start 61.3 37)
+		(end 61.3 37.2)
+		(width 0.2)
+		(layer "F.Cu")
+		(net 6)
+	)
+	(segment
 		(start 60.9 46.9235)
 		(end 60.9 47.189)
@@
 		(net 6)
 	)
+	(via
+		(at 56.5 34.1)
+		(size 0.6)
+		(drill 0.35)
+		(layers "F.Cu" "B.Cu")
+		(net 6)
+	)
+	(via
+		(at 61.3 37)
+		(size 0.6)
+		(drill 0.35)
+		(layers "F.Cu" "B.Cu")
+		(net 6)
+	)
+	(segment
+		(start 58 35.6)
+		(end 56.5 34.1)
+		(width 0.15)
+		(layer "B.Cu")
+		(net 6)
+	)
+	(segment
+		(start 58.3 36.6)
+		(end 58 36.3)
+		(width 0.15)
+		(layer "B.Cu")
+		(net 6)
+	)
+	(segment
+		(start 60.9 36.6)
+		(end 58.3 36.6)
+		(width 0.15)
+		(layer "B.Cu")
+		(net 6)
+	)
+	(segment
+		(start 58 36.3)
+		(end 58 35.6)
+		(width 0.15)
+		(layer "B.Cu")
+		(net 6)
+	)
+	(segment
+		(start 61.3 37)
+		(end 60.9 36.6)
+		(width 0.15)
+		(layer "B.Cu")
+		(net 6)
+	)
 	(segment
 		(start 46.970104 24.8)
@@
 	)
 	(segment
-		(start 59.575 35.382536)
-		(end 55.9 31.707536)
+		(start 51 25.9)
+		(end 52.3 25.9)
 		(width 0.15)
 		(layer "B.Cu")
@@
 	)
 	(segment
-		(start 55.9 31.707536)
-		(end 55.9 29.5)
+		(start 55.7 39.1)
+		(end 56.2 39.6)
 		(width 0.15)
 		(layer "B.Cu")
@@
 	)
 	(segment
-		(start 62.6 46.4)
-		(end 61.357537 46.4)
+		(start 56.2 39.6)
+		(end 58.875 39.6)
 		(width 0.15)
 		(layer "B.Cu")
@@
 	)
 	(segment
-		(start 59.575 44.617463)
-		(end 59.575 35.382536)
+		(start 55.7 29.3)
+		(end 55.7 39.1)
 		(width 0.15)
 		(layer "B.Cu")
@@
 	)
 	(segment
-		(start 51 25.9)
-		(end 52.3 25.9)
+		(start 61.357537 46.4)
+		(end 62.6 46.4)
 		(width 0.15)
 		(layer "B.Cu")
@@
 	)
 	(segment
-		(start 52.3 25.9)
-		(end 55.9 29.5)
+		(start 59.575 44.617463)
+		(end 61.357537 46.4)
 		(width 0.15)
 		(layer "B.Cu")
@@
 	)
 	(segment
-		(start 61.357537 46.4)
+		(start 59.575 40.3)
 		(end 59.575 44.617463)
 		(width 0.15)
 		(layer "B.Cu")
+		(net 21)
+	)
+	(segment
+		(start 58.875 39.6)
+		(end 59.575 40.3)
+		(width 0.15)
+		(layer "B.Cu")
+		(net 21)
+	)
+	(segment
+		(start 52.3 25.9)
+		(end 55.7 29.3)
+		(width 0.15)
+		(layer "B.Cu")
