File: hardware/babelfish.kicad_sch (KiCad schematic)
At the start: 101 parts, among them J2 SWD, J3 DE9 Female, J4 USB_A, Q1 BSS138, SW1 TS342A2P-WZ, SW2 TS342A2P-WZ, U1 RP2040, U11 MAX3232IDR, U12 AP2191WG-7, U2 TPS2113ADRBR, U3 GT-USB-7010ASV, U36 TPS62933, U4 W25Q128JVS, U6 TPMCP1703T-3302E_CB, U7 74HC4052PW,118, U8 74HC4052PW,118, X1 X322512MSB4SI

Commit message: WIP dip switches
Connections:
- net 5V0: now also DIP2.5; no longer DIP2.4
- net VCC_5V: now also DIP2.3; no longer DIP2.6
- net VCC_IN: now also DIP2.6, DIP2.7, DIP2.8; no longer DIP2.1, DIP2.2, DIP2.3
- net VCC_IN_SW: now also DIP2.4; no longer DIP2.5
- net VSHIFT: now also DIP2.1, DIP2.2; no longer DIP2.7, DIP2.8
Other:
- note added: "VCC>5V: 3 on, 4 off VCC=5V: 3 off, 4 on VSHIFT=VCC, 1 off, 2 on VSHIFT=5V, 1 on, 2 off"
- note removed: "VCC>5V: 1 on, 2 off VCC=5V: 1 off, 2 on VSHIFT=VCC, 3 on, 4 off VSHIFT=5V, 3 off, 4 on"
Changed lines of the file:
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@@
   (junction (at 161.29 257.81) (diameter 0) (color 0 0 0 0)
   )
-  (junction (at 302.895 140.97) (diameter 0) (color 0 0 0 0)
+  (junction (at 321.945 148.59) (diameter 0) (color 0 0 0 0)
   )
   (junction (at 177.165 42.545) (diameter 0) (color 0 0 0 0)
@@
   (junction (at 211.455 42.545) (diameter 0) (color 0 0 0 0)
   )
-  (junction (at 322.58 146.05) (diameter 0) (color 0 0 0 0)
+  (junction (at 302.26 143.51) (diameter 0) (color 0 0 0 0)
   )
   (junction (at 291.465 178.435) (diameter 0) (color 0 0 0 0)
@@
     (stroke (width 0) (type default))
   )
-  (wire (pts (xy 322.58 146.05) (xy 331.47 146.05))
+  (wire (pts (xy 302.26 143.51) (xy 293.37 143.51))
     (stroke (width 0) (type default))
   )
@@
     (stroke (width 0) (type default))
   )
-  (wire (pts (xy 302.895 140.97) (xy 302.895 143.51))
+  (wire (pts (xy 321.945 148.59) (xy 321.945 146.05))
     (stroke (width 0) (type default))
   )
@@
     (stroke (width 0) (type default))
   )
-  (wire (pts (xy 320.04 143.51) (xy 331.47 143.51))
+  (wire (pts (xy 304.8 146.05) (xy 293.37 146.05))
     (stroke (width 0) (type default))
   )
@@
     (stroke (width 0) (type default))
   )
-  (wire (pts (xy 292.735 148.59) (xy 304.8 148.59))
+  (wire (pts (xy 332.105 140.97) (xy 320.04 140.97))
     (stroke (width 0) (type default))
   )
@@
     (stroke (width 0) (type default))
   )
-  (wire (pts (xy 292.735 146.05) (xy 304.8 146.05))
+  (wire (pts (xy 332.105 143.51) (xy 320.04 143.51))
     (stroke (width 0) (type default))
   )
@@
     (stroke (width 0) (type default))
   )
-  (wire (pts (xy 320.04 140.97) (xy 331.47 140.97))
+  (wire (pts (xy 304.8 148.59) (xy 293.37 148.59))
     (stroke (width 0) (type default))
   )
@@
     (stroke (width 0) (type default))
   )
-  (wire (pts (xy 322.58 148.59) (xy 320.04 148.59))
+  (wire (pts (xy 302.26 140.97) (xy 304.8 140.97))
     (stroke (width 0) (type default))
   )
@@
     (stroke (width 0) (type default))
   )
-  (wire (pts (xy 292.735 140.97) (xy 302.895 140.97))
+  (wire (pts (xy 332.105 148.59) (xy 321.945 148.59))
     (stroke (width 0) (type default))
   )
@@
     (stroke (width 0) (type default))
   )
-  (wire (pts (xy 302.895 143.51) (xy 304.8 143.51))
+  (wire (pts (xy 321.945 146.05) (xy 320.04 146.05))
     (stroke (width 0) (type default))
   )
@@
     (stroke (width 0) (type default))
   )
-  (wire (pts (xy 320.04 146.05) (xy 322.58 146.05))
+  (wire (pts (xy 304.8 143.51) (xy 302.26 143.51))
     (stroke (width 0) (type default))
   )
@@
     (stroke (width 0) (type default))
   )
-  (wire (pts (xy 322.58 146.05) (xy 322.58 148.59))
+  (wire (pts (xy 302.26 143.51) (xy 302.26 140.97))
     (stroke (width 0) (type default))
   )
@@
     (stroke (width 0) (type default))
   )
-  (wire (pts (xy 304.8 140.97) (xy 302.895 140.97))
+  (wire (pts (xy 320.04 148.59) (xy 321.945 148.59))
     (stroke (width 0) (type default))
   )
@@
     (effects (font (size 1.27 1.27)) (justify left bottom))
   )
-  (text "VCC>5V: 1 on, 2 off\nVCC=5V: 1 off, 2 on\nVSHIFT=VCC, 3 on, 4 off\nVSHIFT=5V, 3 off, 4 on\n"
+  (text "VCC>5V: 3 on, 4 off\nVCC=5V: 3 off, 4 on\nVSHIFT=VCC, 1 off, 2 on\nVSHIFT=5V, 1 on, 2 off\n"
     (at 302.26 160.655 0)
     (effects (font (size 1.27 1.27)) (justify left bottom))
@@
     (effects (font (size 1.27 1.27)) (justify right bottom))
   )
-  (label "VSHIFT" (at 331.47 146.05 180) (fields_autoplaced)
-    (effects (font (size 1.27 1.27)) (justify right bottom))
+  (label "VSHIFT" (at 293.37 143.51 0) (fields_autoplaced)
+    (effects (font (size 1.27 1.27)) (justify left bottom))
   )
   (label "QSPI_SD3" (at 33.02 103.505 0) (fields_autoplaced)
@@
     (effects (font (size 1.27 1.27)) (justify left bottom))
   )
-  (label "VCC_IN" (at 292.735 140.97 0) (fields_autoplaced)
-    (effects (font (size 1.27 1.27)) (justify left bottom))
+  (label "VCC_IN" (at 332.105 148.59 180) (fields_autoplaced)
+    (effects (font (size 1.27 1.27)) (justify right bottom))
   )
   (label "GPIO19" (at 187.325 130.175 180) (fields_autoplaced)
@@
     (effects (font (size 1.27 1.27)) (justify left bottom))
   )
-  (label "5V0" (at 292.735 148.59 0) (fields_autoplaced)
-    (effects (font (size 1.27 1.27)) (justify left bottom))
+  (label "5V0" (at 332.105 140.97 180) (fields_autoplaced)
+    (effects (font (size 1.27 1.27)) (justify right bottom))
   )
   (label "VCC_5V" (at 354.33 107.315 180) (fields_autoplaced)
@@
     (effects (font (size 1.27 1.27)) (justify right bottom))
   )
-  (label "VCC_IN" (at 292.735 146.05 0) (fields_autoplaced)
-    (effects (font (size 1.27 1.27)) (justify left bottom))
+  (label "VCC_IN" (at 332.105 143.51 180) (fields_autoplaced)
+    (effects (font (size 1.27 1.27)) (justify right bottom))
   )
   (label "LED_AUX" (at 187.325 109.855 180) (fields_autoplaced)
@@
     (effects (font (size 1.27 1.27)) (justify left bottom))
   )
-  (label "VCC_IN_SW" (at 331.47 140.97 180) (fields_autoplaced)
-    (effects (font (size 1.27 1.27)) (justify right bottom))
+  (label "VCC_IN_SW" (at 293.37 148.59 0) (fields_autoplaced)
+    (effects (font (size 1.27 1.27)) (justify left bottom))
   )
   (label "TX_A_2Y2" (at 259.08 180.975 0) (fields_autoplaced)
@@
     (effects (font (size 1.27 1.27)) (justify right bottom))
   )
-  (label "VCC_5V" (at 331.47 143.51 180) (fields_autoplaced)
-    (effects (font (size 1.27 1.27)) (justify right bottom))
+  (label "VCC_5V" (at 293.37 146.05 0) (fields_autoplaced)
+    (effects (font (size 1.27 1.27)) (justify left bottom))
   )
   (label "QSPI_SD0" (at 94.615 86.995 0) (fields_autoplaced)

Commit message: v3 rc0
Parts:
- removed C38: 100n, Capacitor_SMD:C_0402_1005Metric, symbol Device:C_Small
- removed C39: 33n, Capacitor_SMD:C_01005_0402Metric, symbol Device:C_Small
- removed C40: 47p, Capacitor_SMD:C_0402_1005Metric, symbol Device:C_Small
- removed C41: 22u, Capacitor_SMD:C_0805_2012Metric, symbol Device:C_Small
- removed DIP2: DSWB04LHGET, lcsc:SW-TH_DSWB04LHGET, symbol LCSC:DSWB04LHGET
- removed L36: 2.7uH, lcsc:IND-SMD_L6.0-W6.0_FNR60XXS, symbol Device:L_Small
- removed R36: 52k3, Resistor_SMD:R_0402_1005Metric, symbol Device:R_Small
- removed R37: 15k, Resistor_SMD:R_0402_1005Metric, symbol Device:R_Small
- removed R38: 10k, Resistor_SMD:R_0402_1005Metric, symbol Device:R_Small
- removed U36: TPS62933, Package_TO_SOT_SMD:SOT-583-8, symbol Regulator_Switching:TPS62933
- removed U7, U8: 74HC4052PW,118, lcsc:TSSOP-16_L5.0-W4.4-P0.65-LS6.4-BL, symbol LCSC:74HC4052PW,118
- added TP11, TP12, TP13, TP14, TP6, TP7, TP8, TP9: TestPoint, TestPoint:TestPoint_Pad_D2.0mm, symbol Connector:TestPoint
- added U7, U8: SN74CBT3253CPWR, lcsc:TSSOP-16_L5.0-W4.4-P0.65-LS6.4-TL, symbol LCSC:SN74CBT3253CPWR
- C36: footprint Capacitor_SMD:C_01005_0402Metric -> Capacitor_SMD:C_0402_1005Metric; ESR 1mOhm -> (none)
- C37: value 10u -> 100n; footprint Capacitor_SMD:C_0805_2012Metric -> Capacitor_SMD:C_0402_1005Metric; ESR 2.8mOhm -> (none)
- TP1, TP2, TP3, TP4, TP5: footprint TestPoint:TestPoint_Pad_D1.0mm -> TestPoint:TestPoint_Pad_D2.0mm
Connections:
- net VCC_IN is gone; now on net VCC_5V: J3.6, TP2.1
- net VCC_IN_SW is gone; now on net GND: C37.1
- net VSHIFT is gone; now on net 5V0: R19.1, R21.1, R23.1, R25.1
- net 5V0: now also C36.2, C37.2, U7.16 (VCC), U8.16 (VCC)
- net CH_A_S0: now also U7.14 (S0)
- net CH_A_S1: now also U7.2 (S1)
- net CH_B_S0: now also U8.14 (S0)
- net CH_B_S1: now also U8.2 (S1)
- net GND: now also C36.1, U7.1 (1OE#), U7.15 (2OE#), U7.8 (GND), U8.1 (1OE#), U8.15 (2OE#), U8.8 (GND); no longer C37.2
- net GPIO14: now also J3.4; no longer J3.5
- net GPIO15: now also J3.5; no longer J3.4
- net RX_A: now also TP12.1, U7.7 (1A)
- net RX_A_CONN: now also TP7.1, U7.6 (1B1)
- net RX_B: now also TP14.1, U8.7 (1A)
- net RX_B_CONN: now also TP9.1, U8.6 (1B1)
- net TX_A: now also TP11.1, U7.9 (2A)
- net TX_A_CONN: now also TP6.1, U7.10 (2B1)
- net TX_B: now also TP13.1, U8.9 (2A)
- net TX_B_CONN: now also TP8.1, U8.10 (2B1)
- net RX_A_1Y1 renamed RX_A_SHIFTER
- net RX_A_SHIFTER: now also U7.5 (1B2)
- net RX_A_1Y2 renamed RX_A_MAX
- net RX_A_MAX: now also U7.4 (1B3)
- net RX_A_2Y1 renamed RX_A_SHIFTER_OUT
- net RX_A_2Y2 renamed RX_A_MAX_OUT
- net RX_B_1Y1 renamed RX_B_SHIFTER
- net RX_B_SHIFTER: now also U8.5 (1B2)
- net RX_B_1Y2 renamed RX_B_MAX
- net RX_B_MAX: now also U8.4 (1B3)
- net RX_B_2Y1 renamed RX_B_SHIFTER_OUT
- net RX_B_2Y2 renamed RX_B_MAX_OUT
- net TX_A_1Y1 renamed TX_A_SHIFTER
- net TX_A_SHIFTER: now also U7.11 (2B2)
- net TX_A_1Y2 renamed TX_A_MAX
- net TX_A_MAX: now also U7.12 (2B3)
- net TX_A_2Y1 renamed TX_A_SHIFTER_OUT
- net TX_A_2Y2 renamed TX_A_MAX_OUT
- net TX_B_1Y1 renamed TX_B_SHIFTER
- net TX_B_SHIFTER: now also U8.11 (2B2)
- net TX_B_1Y2 renamed TX_B_MAX
- net TX_B_MAX: now also U8.12 (2B3)
- net TX_B_2Y1 renamed TX_B_SHIFTER_OUT
- net TX_B_2Y2 renamed TX_B_MAX_OUT
- no-connect marks 17 -> 16
Other:
- note added: "Power notes: Tagged as power: VBUS - incoming 5V USB power VCC_5V - incoming 5V from DB9 Internal routing: 3V3 - 3.3v supply 5V0 - 5v supply (either VBUS or VCC_5V) current limited to 357mA @ TPS2113 VBUS_OUT - outgoing 5V USB power."
- note added: "Test Points"
- note removed: "5v0 Power (from VCC)"
- note removed: "Power notes: Tagged as power: VBUS - incoming 5V USB power VCC_IN - incoming VCC from connector (5V-12V) Internal routing: VCC_IN_SW - VCC incoming that goes TPS62933 VCC_5V - VCC converted to 5V 3V3 - 3.3v supply 5V0 - 5v supply current limited to 357mA @ TPS2113 VBUS_OUT - outgoing 5V USB power."
- note removed: "VCC>5V: 3 on, 4 off VCC=5V: 3 off, 4 on VSHIFT=VCC, 1 off, 2 on VSHIFT=5V, 1 on, 2 off"
- moved on the sheet: TP1, TP2, TP3, TP4, TP5
